File: KiCad/apple-color-monitor-iie-a2m2056/apple-color-monitor-iie-a2m2056.kicad_sch (KiCad schematic)
At the start: 395 parts, among them CN14 Conn_01x04_Pin, CN16 Conn_01x01_Pin, CN20 Conn_01x06_Pin, CN20_plug1 Conn_01x06, CN4 Conn_01x07_Pin, CN4_FRONT1 CN, CN5 Text/Gfx, CN5_FRONT1 Conn_01x02_Socket, CN6 GRN, CN8 Conn_01x02_Pin, CN9 Conn_01x01_Pin, IC102 CD4053B, J101 Jumper_2_Bridged, J102 Jumper_2_Bridged, J103 Jumper_2_Bridged, J104 Jumper_2_Bridged, J106 Jumper_2_Bridged, J107 Jumper_2_Bridged, J108 Jumper_2_Bridged, J109 Jumper_2_Bridged, J110 Jumper_2_Bridged, J111 Jumper_2_Bridged, J112 Jumper_2_Bridged, J113 Jumper_2_Bridged, J114 Jumper_2_Bridged, J126 Jumper_2_Bridged, J201 Jumper_2_Bridged, J202 Jumper_2_Bridged, J203 Jumper_2_Bridged, J204 Jumper_2_Bridged, J205 Jumper_2_Bridged, J302 Jumper_2_Bridged, J304 Jumper_2_Bridged, J306 Jumper_2_Bridged, J308 Jumper_2_Bridged, J401 Jumper_2_Bridged, J402 Jumper_2_Bridged, J603 Jumper_2_Bridged, J604 Jumper_2_Bridged, J801 Jumper_2_Bridged, J802 Jumper_2_Bridged, J803 Jumper_2_Bridged, J804 Jumper_2_Bridged, J805 Jumper_2_Bridged, J806 Jumper_2_Bridged, P701 VIDEO IN, Q101 C945, Q102 A733, Q103 A733, Q104 C945, Q105 A733, Q111 A642, Q114 C945, Q201 C1507, Q202 D1398, Q501 A709, Q502 C1008, Q503 C3042, Q504 A709, Q801 C945, Q802 C945, Q803 C945, Q804 A733, Q805 A733, Q806 A733, Q807 A733, Q808 A733, Q809 A733, SW1 SW_SPST, SW800 SVC_SW, T102 Transformer_1P_1S, T103 Transformer_1P_1S, T201 Transformer_1P_1S, T202 Transformer_1P_1S, T203 Transformer_SP_2S, T204 Fkyback, T205 Transformer_1P_1S, T501 Transformer_4_5_Unknwon, X102 DL401F5, X103 Crystal

Commit message: checkpoint
Parts:
- Q202: symbol Transistor_BJT:Q_NPN_BCE -> -my-symbols:_Power_Transistor_NPN_D1398
Other:
- moved on the sheet: C104, C105, C106, C112, C222, C223, C224, C225, C226, C229, C230, C502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

Commit message: checkpoint
Connections:
- net at V_YOKE1.1: now also CN20_plug1.2 (GRN); no longer CN20_plug1.1 (YLW)
- net at V_YOKE1.2: now also CN20_plug1.1 (YLW); no longer CN20_plug1.2 (GRN)
Other:
- moved on the sheet: H_YOKE1, V_YOKE1
Changed lines of the file:
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@@
 	(text_box "ISOLATED"
 		(exclude_from_sim no)
-		(at 801.37 504.825 0)
+		(at 805.18 504.825 0)
 		(size 6.35 1.905)
 		(margins 0.127 0.127 0.127 0.127)
@@
 	(text_box "LIVE"
 		(exclude_from_sim no)
-		(at 802.64 543.4686 0)
+		(at 806.45 543.4686 0)
 		(size 5.08 2.6314)
 		(margins 0.127 0.127 0.127 0.127)
@@
 	(wire
 		(pts
-			(xy 814.07 538.48) (xy 814.07 551.18)
+			(xy 817.88 538.48) (xy 817.88 551.18)
 		)
 		(stroke
@@
 	(wire
 		(pts
-			(xy 806.45 500.38) (xy 801.37 500.38)
+			(xy 810.26 500.38) (xy 805.18 500.38)
 		)
 		(stroke
@@
 	(wire
 		(pts
-			(xy 814.07 500.38) (xy 814.07 513.08)
+			(xy 817.88 500.38) (xy 817.88 513.08)
 		)
 		(stroke
@@
 	(wire
 		(pts
-			(xy 814.07 513.08) (xy 801.37 513.08)
+			(xy 817.88 513.08) (xy 805.18 513.08)
 		)
 		(stroke
@@
 	(wire
 		(pts
-			(xy 814.07 551.18) (xy 801.37 551.18)
+			(xy 817.88 551.18) (xy 805.18 551.18)
 		)
 		(stroke
@@
 	(wire
 		(pts
-			(xy 801.37 538.48) (xy 806.45 538.48)
+			(xy 805.18 538.48) (xy 810.26 538.48)
 		)
 		(stroke
@@
 	(symbol
 		(lib_id "Device:L")
-		(at 810.26 538.48 90)
+		(at 814.07 538.48 90)
 		(unit 1)
 		(body_style 1)
@@
 		(fields_autoplaced yes)
 		(property "Reference" "H_YOKE1"
-			(at 810.26 535.94 90)
+			(at 814.07 535.94 90)
 			(show_name no)
 			(do_not_autoplace no)
@@
 		)
 		(property "Value" "L"
-			(at 811.5299 537.21 0)
+			(at 815.3399 537.21 0)
 			(hide yes)
 			(show_name no)
@@
 		)
 		(property "Footprint" ""
-			(at 810.26 538.48 0)
+			(at 814.07 538.48 0)
 			(hide yes)
 			(show_name no)
@@
 		)
 		(property "Datasheet" ""
-			(at 810.26 538.48 0)
+			(at 814.07 538.48 0)
 			(hide yes)
 			(show_name no)
@@
 		)
 		(property "Description" "Inductor"
-			(at 810.26 538.48 0)
+			(at 814.07 538.48 0)
 			(hide yes)
 			(show_name no)
@@
 	(symbol
 		(lib_id "Connector:Conn_01x06_Pin")
-		(at 789.94 525.78 0)
-		(mirror y)
+		(at 787.4 525.78 0)
 		(unit 1)
 		(body_style 1)
@@
 		)
 		(property "Value" "Conn_01x06_Pin"
-			(at 789.305 517.398 0)
+			(at 788.035 517.398 0)
 			(hide yes)
 			(show_name no)
@@
 		)
 		(property "Footprint" "_my-footprints:_CN20_pins"
-			(at 789.94 525.78 0)
+			(at 787.4 525.78 0)
 			(hide yes)
 			(show_name no)
@@
 		)
 		(property "Description" "Generic connector, single row, 01x06, script generated"
-			(at 789.94 525.78 0)
+			(at 787.4 525.78 0)
 			(hide yes)
 			(show_name no)
@@
 	(symbol
 		(lib_id "Device:L")
-		(at 810.26 500.38 90)
+		(at 814.07 500.38 90)
 		(unit 1)
 		(body_style 1)
@@
 		(fields_autoplaced yes)
 		(property "Reference" "V_YOKE1"
-			(at 810.26 497.84 90)
+			(at 814.07 497.84 90)
 			(show_name no)
 			(do_not_autoplace no)
@@
 		)
 		(property "Value" "L"
-			(at 811.5299 499.11 0)
+			(at 815.3399 499.11 0)
 			(hide yes)
 			(show_name no)
@@
 		)
 		(property "Footprint" ""
-			(at 810.26 500.38 0)
+			(at 814.07 500.38 0)
 			(hide yes)
 			(show_name no)
@@
 		)
 		(property "Datasheet" ""
-			(at 810.26 500.38 0)
+			(at 814.07 500.38 0)
 			(hide yes)
 			(show_name no)
@@
 		)
 		(property "Description" "Inductor"
-			(at 810.26 500.38 0)
+			(at 814.07 500.38 0)
 			(hide yes)
 			(show_name no)
@@
 	(symbol
 		(lib_id "Connector_Generic:Conn_01x06")
-		(at 796.29 525.78 0)
-		(mirror y)
+		(at 802.64 525.78 0)
 		(unit 1)
 		(body_style 1)
@@
 		(dnp no)
 		(property "Reference" "CN20_plug1"
-			(at 798.576 519.176 90)
+			(at 802.386 519.176 90)
 			(show_name no)
 			(do_not_autoplace no)
@@
 		)
 		(property "Value" "Conn_01x06"
-			(at 796.29 516.89 0)
+			(at 802.64 516.89 0)
 			(hide yes)
 			(show_name no)
@@
 		)
 		(property "Footprint" ""
-			(at 796.29 525.78 0)
+			(at 800.1 525.78 0)
 			(hide yes)
 			(show_name no)
@@
 		)
 		(property "Datasheet" ""
-			(at 796.29 525.78 0)
+			(at 800.1 525.78 0)
 			(hide yes)
 			(show_name no)
@@
 		)
 		(property "Description" "Generic connector, single row, 01x06, script generated (kicad-library-utils/schlib/autogen/connector/)"
-			(at 796.29 525.78 0)
+			(at 802.64 525.78 0)
 			(hide yes)
 			(show_name no)

Commit message: checkpoint
Parts:
- added D509: D, Diode_THT:D_DO-15_P12.70mm_Horizontal, symbol Device:D
Connections:
- net FLY_7: now reaches T204.7, T205.3 (SA)
- net FLY_7: now also D509.2 (A); no longer D502.2 (A)
- net FLY_7_D: no longer names the net of C516.2, R503.2
- net FLY_7_D: now also D509.1 (K); no longer D502.1 (K)
Other:
- moved on the sheet: C502, C503, C504, C505, C506, C512, C516, CN9, D501, D502, D503, D504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

Commit message: checkpoint
Parts:
- removed D509: D, Diode_THT:D_DO-15_P12.70mm_Horizontal, symbol Device:D
Connections:
- net FLY_7: now also D502.2 (A)
- net at C516.2, R503.2: now also D502.1 (K)
- net FLY_14_R renamed FLY_13_R
Other:
- moved on the sheet: C305, C308, C502, C503, C504, C505, C506, C512, C516, CN9, D104, D301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

Commit message: checkpoint
Parts:
- added C901, C902, C903, C904, C905, C906: C_Small, _my-footprints:_C_Axial_P5.0mm, symbol Device:C_Small
- added C907: C_Small, Resistor_THT:R_Axial_DIN0204_L3.6mm_D1.6mm_P7.62mm_Horizontal, symbol Device:C_Small
- added C908: C, Capacitor_THT:CP_Radial_D8.0mm_P5.00mm, symbol Device:C_Polarized
- added CN42: (no value), _my-footprints:-crt-neck, symbol -my-symbols:-crt-neck-connector
- added JP901: Jumper_2_Bridged, _my-footprints:_Jumper_4mm, symbol Jumper:Jumper_2_Bridged
- added L902, L903: L, _my-footprints:_L_Axial_P5.0mm, symbol Device:L
- added NECK_CN14: Conn_01x04_Socket, Connector_Molex:Molex_KK-254_AE-6410-04A_1x04_P2.54mm_Vertical, symbol Connector:Conn_01x04_Socket
- added NECK_CN16: Conn_01x01_Pin, Connector_Pin:Pin_D1.0mm_L10.0mm, symbol Connector:Conn_01x01_Pin
- added NECK_CN8: Conn_01x02_Pin, Connector_Wire:SolderWire-0.127sqmm_1x02_P3.7mm_D0.48mm_OD1mm, symbol Connector:Conn_01x02_Pin
- added NECK_E1: Conn_01x01_Pin, _my-footprints:-SolderWire, symbol Connector:Conn_01x01_Pin
- added NECK_SH1: RFShield_OnePiece, RF_Shielding:Laird_Technologies_BMI-S-103_26.21x26.21mm, symbol Device:RFShield_OnePiece
- added Q901, Q902, Q903: C1507, _my-footprints:-TO-220-3_Vertical-BCE_FIN, symbol Transistor_BJT:Q_NPN_BCE
- added Q904, Q905, Q906: C2330, _my-footprints:-Transistor_ECB-NPN, symbol Transistor_BJT:Q_NPN_ECB
- added R901, R902, R903, R904, R905, R906, R907, R908, R909, R910, R911, R912: R, Resistor_THT:R_Axial_DIN0207_L6.3mm_D2.5mm_P10.16mm_Horizontal, symbol Device:R
- added R913, R914, R915: R, _my-footprints:R_Axial_side_shift_P20.32mm, symbol Device:R
- added R916, R918, R920, R921, R922, R923: R, Resistor_THT:R_Axial_DIN0309_L9.0mm_D3.2mm_P12.70mm_Horizontal, symbol Device:R
- added R917: R, Resistor_THT:R_Axial_DIN0207_L6.3mm_D2.5mm_P15.24mm_Horizontal, symbol Device:R
- Q503: footprint Package_TO_SOT_THT:TO-3P-3_Vertical -> _my-footprints:_TO-3P-3_Vertical_BCE
- renumbered R901 to R701, R902 to R702
Connections:
- net GNDPWR: now also TP_GNDPWR1.TP (TP_GNDPWR); no longer TP_GNDPWR1.1 (Pin_1)
- net at C509.1, Q502.3 (C), Q503.2 (C)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: now also L502.1; no longer R504.1
- net at C508.1, D506.2 (A), T501.5 (PC): now also L502.2; no longer L502.1
- net at R919.2, R924.2: now also CN8.2 (H); no longer CN8.H (Pin_2)
- net at C140.1, D107.1 (K): now also CN8.1 (B); no longer CN8.B (Pin_1)
- net at Q503.1 (B): now also R504.1; no longer L502.2
- new net: C906.2, Q906.1 (E), R912.2
- new net: Q903.3 (E), Q906.2 (C)
- new net: Q906.3 (B), R909.2
- new net: C907.1, CN42.7 (S)
- new net: C907.2, CN42.2 (G), CN42.3 (G), CN42.5 (G), CN42.9 (H), NECK_CN16.1 (Pin_1)
- new net: NECK_CN8.2 (H), R923.1
- new net: CN42.10 (H), R923.2
- new net: JP901.1 (A), R913.2, R920.2
- new net: JP901.2 (B), Q901.2 (C), R916.1
- new net: C905.1, Q905.1 (E), R911.2
- new net: L902.2, R914.2, R921.1
- new net: CN42.6 (GK), R917.1
- new net: L902.1, Q902.2 (C), R917.2
- new net: C901.1, Q901.1 (B), R901.1, R904.2
- new net: NECK_CN14.3 (B), R909.1
- new net: C903.1, Q903.1 (B), R903.2, R906.1
- new net: C902.1, Q902.1 (B), R902.2, R905.2
- new net: NECK_CN14.1 (R), R907.1
- new net: Q904.3 (B), R907.2
- new net: C904.1, Q904.1 (E), R910.2
- new net: Q901.3 (E), Q904.2 (C)
- new net: L903.1, R915.1, R922.2
- new net: L903.2, Q903.2 (C), R918.1
- new net: NECK_CN14.2 (G), R908.2
- new net: Q902.3 (E), Q905.2 (C)
- new net: Q905.3 (B), R908.1
- new net: CN42.8 (RK), R916.2
- new net: CN42.11 (BK), R918.2
- new net NECK_B: C908.1, NECK_CN8.1 (B), R901.2, R902.1, R903.1, R913.1, R914.1, R915.2, R920.1, R921.2, R922.1
- new net NECK_E: C901.2, C902.2, C903.2, C904.2, C905.2, C906.1, C908.2, NECK_CN14.4 (E), NECK_E1.1 (Pin_1), NECK_SH1.1 (Shield), R904.1, R905.1, R906.2, R910.1, R911.1, R912.1
Other:
- note added: "-10V 100VAC"
- note added: "-10V 101VAC"
- note added: "-2.0V 1.9VAC"
- note added: "-2.3V 1.3VAC"
- note added: "-2V 1.8VAC"
- note added: "-3V"
- note added: "-68V"
- note added: "-75V 61VAC"
- note added: "-77V"
- note added: "-78V"
- note added: "-78V 61VAC"
- note added: "-9V"
- note added: "-9V 60VAC"
- note added: "-9V 61VAC"
- note added: "0.1V"
- note added: "0.3V"
- note added: "0.5V"
- note added: "0.6V"
- note added: "0.6V 6.1VAC"
- note added: "0.7V"
- note added: "0.9V 2VAC"
- note added: "0.9V 8.4VAC"
- note added: "0V"
- note added: "0V 44.8VAC"
- note added: "0V 45VAC"
- note added: "0V 53VAC"
- note added: "0V 5AC"
- note added: "0V 6.3VAC"
- note added: "0V 6.4VAC"
- note added: "0V 60VAC"
- note added: "0V 9.0VAC"
- note added: "0VAC"
- note added: "1.0V"
- note added: "1.1V"
- note added: "1.1V 1.7VAC"
- note added: "1.2V"
- note added: "1.3V"
- note added: "1.4V"
- note added: "1.5V"
- note added: "1.8V 4.0VAC"
- note added: "108V 1670VAC"
- note added: "108V 60VAC"
- note added: "11 - 12 53VAC 12 - 13 46VAC 13 - 14 3VAC 14 - 15 34VAC 15 - 16 24VAC 11 - 13 6.7VAC 11 - 14 0.7VAC 11 - 15 45VAC 11 - 16 60VAC 12 - 14 59VAC 12 - 15 82VAC 12 - 16 94VAC 13 - 15 49VAC 14 - 16 57VAC 14 - 16 45VAC"
- note added: "11.0V"
- note added: "11.2V 8.8VAC"
- note added: "11.2VAC"
- note added: "12.2V"
- note added: "12.3V"
- note added: "12.4V"
- note added: "12.5V"
- note added: "12.7V"
- note added: "12.8V"
- note added: "12.9V"
- note added: "121VAC"
- note added: "13.0V"
- note added: "13.3V"
- note added: "13.4V"
- note added: "158V"
- note added: "17.3V"
- note added: "17.6V"
- note added: "17.6V 0.7VAC"
- note added: "1793VAC"
- note added: "18.4V"
- note added: "187V"
- note added: "187V 0VAC"
- note added: "2.1V 1.4VAC"
- note added: "24.9V"
- note added: "26.1V"
- note added: "26.3V"
- note added: "26.5V"
- note added: "28.1V"
- note added: "3.4V"
- note added: "3.6V"
- note added: "31.6VAC"
- note added: "31V 80VAC"
- note added: "32.6V 2.5VAC"
- note added: "32V 60VAC"
- note added: "4.3V"
- note added: "4.4V"
- note added: "4.5V"
- note added: "4.6VAC"
- note added: "4.7V"
- note added: "4.7V 0.6VAC"
- note added: "4.9V"
- note added: "44.8VAC"
- note added: "45VAC"
- note added: "46VAC"
- note added: "5.1V"
- note added: "6.1VAC"
- note added: "6.3V"
- note added: "7 - 7.5 6VAC 7.5 - 8 45VAC 8 - 9 55VAC 9 - 10 1693VAC 7 - 8 33VAC 7 - 9 9VAC 8 - 10 879VAC 7.5 - 10 1691VAC 7 - 10 1632VAC"
- note added: "7.3V"
- note added: "7.8V"
- note added: "7.9V"
- note added: "71.5V"
- note added: "71V"
- note added: "79V"
- note added: "79V 60VAC"
- note added: "79V 61VAC"
- note added: "8.0V"
- note added: "8.2V"
- note added: "8.4V"
- note added: "8.5V"
- note added: "8.9V"
- note added: "80V 61VAC"
- note added: "88.7V"
- note added: "9.0V"
- note added: "9.2V"
- note added: "9.6VAC"
- note added: "PWB-CRT SOCKET NECK BOARD"
- moved on the sheet: C109, C205, C207, C208, C209, C210, C211, C218, C222, C223, C224, C227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

Commit message: checkpoint
Parts:
- removed CRT_FOCUS1: Conn_01x01_Pin, symbol Connector:Conn_01x01_Pin
- added CRT1: Conn_01x12_Pin, symbol Connector:Conn_01x12_Pin
- G_CN9: renamed from CN6; value GRN -> Conn_01x01_Pin
- NECK_S1: renamed from CRT_SCREEN1; footprint (none) -> _my-footprints:-SolderWire
- renumbered JP901 to J901
Connections:
- net FOCUS: now also CN42.1 (FOCUS)
- net GNDREF: now also C907.2
- net SCREEN: now also C907.1, CN42.7 (S)
- net GND1: now reaches CN42.2 (G), CN42.3 (G), CN42.5 (G), CN42.9 (H), NECK_CN16.1 (Pin_1)
- net GND1: no longer C907.2
- net GK: now reaches CN42.6 (GK), R917.1
- net FLY_16: now reaches R236.1, T204.16
- net RK: now reaches CN42.8 (RK), R916.2
- net BK: now reaches CN42.11 (BK), R918.2
- net FLY_16_RD: no longer names the net of C309.1, D204.1 (K), JP301.2 (B)
Other:
- note added: "7 - 7.5 6VAC 7.5 - 8 45VAC 7.5 - 9 3VAC 8 - 9 55VAC 9 - 10 1207VAC 7 - 8 33VAC 7 - 9 9VAC 8 - 10 739VAC 7.5 - 10 1208VAC 7 - 10 1174VAC"
- note removed: "7 - 7.5 6VAC 7.5 - 8 45VAC 8 - 9 55VAC 9 - 10 1693VAC 7 - 8 33VAC 7 - 9 9VAC 8 - 10 879VAC 7.5 - 10 1691VAC 7 - 10 1632VAC"
- moved on the sheet: C121, C124, C125, C126, C127, C128, C140, C153, C216, C219, C220, C309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

Commit message: checkpoint
Parts:
- added NT1, NT2, NT3, NT4: NetTie, symbol Device:NetTie_2
Connections:
- net NECK_E is gone; now on net GND1: C901.2, C902.2, C903.2, C904.2, C905.2, C906.1, C908.2, NECK_CN14.4 (E), NECK_E1.1 (Pin_1), NECK_SH1.1 (Shield), R904.1, R905.1, R906.2, R910.1, R911.1, R912.1
- net ANODE: now also NT3.1; no longer CRT_ANODE1.1 (Pin_1)
- net FOCUS: now also NT2.1; no longer CN42.1 (FOCUS)
- net GND1: now also C907.2, NT1.2
- net GNDREF: now also NT1.1; no longer C907.2
- net SCREEN: now also NT4.1; no longer C907.1, CN42.7 (S), NECK_S1.1 (S)
- new net: C907.1, CN42.7 (S), NECK_S1.1 (S), NT4.2
- new net: CN42.1 (FOCUS), NT2.2
- new net: CRT_ANODE1.1 (Pin_1), NT3.2
Other:
- company: Apple Computer -> Reverse engineered by Fred Sauer, 2026. Published under Apache 2 license.
- moved on the sheet: C102, C103, C104, C105, C106, C109, C110, C111, C112, C114, C115, C117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

Commit message: checkpoint
Connections:
- net FLY_13: now reaches R161.2, R919.1, R924.1, T204.13
- net H: now reaches CN8.2 (H), R919.2, R924.2
- net B: now reaches C140.1, CN8.1 (B), D107.1 (K)
- net FLY_13_R: no longer names the net of R162.2, VR303.1
Other:
- note added: "0V 5VAC"
- note removed: "-2V 1.8VAC"
- note removed: "0V 5AC"
- moved on the sheet: C140, C161, C302, CN8, D160, R161, R162, R919, R924
