File: KiCad/apple-color-monitor-iie-a2m2056/apple-color-monitor-iie-a2m2056.kicad_sch (KiCad schematic)
At the start: 444 parts, among them CN14 Conn_01x04_Pin, CN16 Conn_01x01_Pin, CN20 Conn_01x06_Pin, CN20_plug1 Conn_01x06, CN4 Conn_01x07_Pin, CN4_FRONT1 CN, CN5 Text/Gfx, CN5_FRONT1 Conn_01x02_Socket, CN8 Conn_01x02_Pin, CN9 Conn_01x01_Pin, IC102 CD4053B, J101 Jumper_2_Bridged, J102 Jumper_2_Bridged, J103 Jumper_2_Bridged, J104 Jumper_2_Bridged, J106 Jumper_2_Bridged, J107 Jumper_2_Bridged, J108 Jumper_2_Bridged, J109 Jumper_2_Bridged, J110 Jumper_2_Bridged, J111 Jumper_2_Bridged, J112 Jumper_2_Bridged, J113 Jumper_2_Bridged, J114 Jumper_2_Bridged, J126 Jumper_2_Bridged, J201 Jumper_2_Bridged, J202 Jumper_2_Bridged, J203 Jumper_2_Bridged, J204 Jumper_2_Bridged, J205 Jumper_2_Bridged, J302 Jumper_2_Bridged, J304 Jumper_2_Bridged, J306 Jumper_2_Bridged, J308 Jumper_2_Bridged, J401 Jumper_2_Bridged, J402 Jumper_2_Bridged, J603 Jumper_2_Bridged, J604 Jumper_2_Bridged, J801 Jumper_2_Bridged, J802 Jumper_2_Bridged, J803 Jumper_2_Bridged, J804 Jumper_2_Bridged, J805 Jumper_2_Bridged, J806 Jumper_2_Bridged, J901 Jumper_2_Bridged, P701 VIDEO IN, Q101 C945, Q102 A733, Q103 A733, Q104 C945, Q105 A733, Q111 A642, Q114 C945, Q201 C1507, Q202 D1398, Q501 A709, Q502 C1008, Q503 C3042, Q504 A709, Q801 C945, Q802 C945, Q803 C945, Q804 A733, Q805 A733, Q806 A733, Q807 A733, Q808 A733, Q809 A733, Q901 C1507, Q902 C1507, Q903 C1507, Q904 C2330, Q905 C2330, Q906 C2330, SW1 SW_SPST, SW800 SVC_SW, T102 Transformer_1P_1S, T103 Transformer_1P_1S, T201 Transformer_1P_1S, T202 Transformer_1P_1S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

Commit message: checkpoint
Parts:
- removed C215: C_Small, Resistor_THT:R_Axial_DIN0204_L3.6mm_D1.6mm_P5.08mm_Horizontal, symbol Device:C_Small
- removed J126: Jumper_2_Bridged, _my-footprints:_Jumper_11mm, symbol Jumper:Jumper_2_Bridged
- added C215: C, Capacitor_THT:CP_Radial_Tantal_D4.5mm_P5.00mm, symbol Device:C_Polarized_Small_US
- added R126: R, Resistor_THT:R_Axial_DIN0309_L9.0mm_D3.2mm_P12.70mm_Horizontal, symbol Device:R
- C908: footprint Capacitor_THT:CP_Radial_D8.0mm_P5.00mm -> _my-footprints:CP_Radial_D5.0mm_P5.00mm
- R921: footprint Resistor_THT:R_Axial_DIN0309_L9.0mm_D3.2mm_P12.70mm_Horizontal -> _my-footprints:R_Axial_P11.0mm
- T102: symbol Device:Transformer_1P_1S -> -my-symbols:_Transformer_5pin
- T103: symbol Device:Transformer_1P_1S -> -my-symbols:_Transformer_7pin
- renumbered C153 to C123, C551 to C221, L207 to L101, R311 to R304
Connections:
- net ACC_FILTER: no longer R125.1
- net GNDREF: now also C215.2
- net KILLER_FILTER: now also R125.1
- net VIDEO_INV_IN: no longer D105.2 (A)
- net VIDEO_INV_OUT: now also D105.2 (A)
- net at C509.1, Q502.3 (C), R503.1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: now also Q503.1 (B), R504.1; no longer L502.1, Q503.2 (C)
- net at C508.1, D506.2 (A), T501.5 (PC): now also L502.1; no longer L502.2
- net H_YOKE: now reaches C225.2, C226.2, CN20.6 (RED), JP501.1 (A), Q202.2 (C)
- net +18.4V: now reaches C138.1, D203.1 (K), R152.1, R168.1, R173.2, R306.2
- net at CN4.2 (PNK): now also R126.2
- net at VR103.1: now also R126.1
- net at IC101.28 (RAMP_CAPACITOR): now also C215.1
- net CONTRAST renamed CONTRAST_OUT_C
- new net: L502.2, Q503.2 (C)
Other:
- note added: "TODO: 18.4 ==> 16V??"
- note added: "TODO: Define Z ?"
- note added: "TODO: Here GRDPWR//GND_COM ??"
- note added: "TODO: Is this 24V?"
- note added: "TODO: Is this Z horizontal?"
- note added: "TODO: Measure voltages around B+ ADJ"
- note added: "TODO: Measure voltages due to 1) color knob, 2) text switch"
- note added: "TODO: Renumber PINS??"
- note added: "TODO: Zener?"
- note added: "TODO: describe as +170V ??"
- note added: "TODO: describe as +50V ??"
- note added: "TODO: verify voltages"
- note removed: "0V 6.3VAC"
- note removed: "1793VAC"
- note removed: "45VAC"
- moved on the sheet: C101, C102, C103, C104, C105, C106, C107, C109, C110, C111, C112, C114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

Commit message: checkpoint
Parts:
- C502, C503, C504, C505: value SAFETY Y -> 'Y'
Connections:
- net CHROMA_OUT: now reaches C122.1, IC101.12 (CHROMA_OUT), TP12.1 (Pin_1)
- net CONTRAST_OUT_E: now reaches C114.1, IC101.2 (CONT.OUT(E)), R130.1
- net DEMO_IN: now reaches C122.2, IC101.14 (DEMO_IN)
- net FLY_13: no longer names the net of R161.2, R919.1, R924.1, T204.13
- net FLY_16: no longer names the net of R236.1, T204.16
- net H_YOKE: no longer names the net of C225.2, C226.2, CN20.6 (RED), JP501.1 (A), Q202.2 (C)
Other:
- note added: "-0.1V 4VAC"
- note added: "-0.2V 23VAC"
- note added: "-0.2V 30VAC 15.7kHz"
- note added: "-0.2V 6VAC"
- note added: "-0.5V 222VAC 15.7kHZ"
- note added: "-0.8V 33VAC 60Hz sawtooth"
- note added: "-0V 24VAC 15.7kHZ"
- note added: "-0V 28VAC 20kHZ"
- note added: "-1.5V 170VAC ~16kHz"
- note added: "-12V 180VAC"
- note added: "-14.5V 344VAC 11.5kHz"
- note added: "-1V 144VAC"
- note added: "-1V 46VAC"
- note added: "-2.2V 10.4VAC"
- note added: "-2.5V 6.6VAC"
- note added: "-3.4V 244VAC 19-20kHZ"
- note added: "-4.6V 184VAC"
- note added: "-5.0V 184VAC"
- note added: "-5V 170VAC 31.4kHz"
- note added: "-71V 184VAC"
- note added: "-75V 180VAC 60Hz"
- note added: "-77.5V 188VAC"
- note added: "-78V 208VAC 60Hz"
- note added: "-80.5V 188VAC"
- note added: "-80V 180VAC"
- note added: "-80V 180VAC 60Hz"
- note added: "-80V 184VAC"
- note added: "0.2V 4VAC"
- note added: "0.3V 1.9VAC"
- note added: "0.3V 2.2VAC"
- note added: "0.6V 2.3VAC"
- note added: "0.8V 17.6VAC 60Hz"
- note added: "0.8V 8.4VAC"
- note added: "0V 29.6VAC 60Hz sawtooth"
- note added: "1.1V 8VAC"
- note added: "1.2V 2.2VAC"
- note added: "1.3V 2.3VAC"
- note added: "1.5V 2.6VAC"
- note added: "1.5V 30VAC 60Hz"
- note added: "105V 188VAC 60Hz"
- note added: "105V 268VAC"
- note added: "105V 300VAC"
- note added: "106V 440VAC 60Hz + 15.7kHz"
- note added: "115V >900VAC 15.7kHz"
- note added: "12.3V 6VAC"
- note added: "12.6V 2VAC"
- note added: "12.8V 2VAC"
- note added: "13.3V 2VAC"
- note added: "17V 4VAC"
- note added: "24.4V 8VAC"
- note added: "26.7V 32VAC 60Hz"
- note added: "29.1V 16VAC"
- note added: "3.3V 11.2VAC"
- note added: "3.5V 3.6VAC"
- note added: "3.6V 6VAC"
- note added: "4.3V 3.6VAC"
- note added: "4.4V 4VAC"
- note added: "4.8V 188VAC"
- note added: "68.4V 188VAC"
- note added: "68V 188VAC"
- note added: "69.1V 188VAC"
- note added: "69V 188VAC"
- note added: "7.6V 2VAC"
- note added: "7.7V 2VAC"
- note added: "76V 188VAC"
- note added: "8.0V 2VAC"
- note added: "8.2V 4.8VAC"
- note added: "8.2V 7.8VAC 60Hz+15kHz"
- note added: "8.3V 8.8VAC"
- note added: "8.4V 8.4VAC 60Hz+15kHz"
- note added: "Chroma / luminance"
- note added: "Composite video in"
- note added: "Deflection"
- note added: "Jumper sandbox"
- note added: "SERVICE SWITCH"
- note added: "Signal processing"
- note added: "X-ray protection"
- note removed: "-10V 100VAC"
- note removed: "-10V 101VAC"
- note removed: "-2.0V 1.9VAC"
- note removed: "-2.3V 1.3VAC"
- note removed: "-3V"
- note removed: "-68V"
- note removed: "-75V 61VAC"
- note removed: "-77V"
- note removed: "-78V"
- note removed: "-78V 61VAC"
- note removed: "-9V"
- note removed: "0.1V"
- note removed: "0.6V 6.1VAC"
- note removed: "0.9V 2VAC"
- note removed: "0.9V 8.4VAC"
- note removed: "0V 44.8VAC"
- note removed: "0V 45VAC"
- note removed: "0V 53VAC"
- note removed: "0V 6.4VAC"
- note removed: "0V 60VAC"
- note removed: "0VAC"
- note removed: "1.0V"
- note removed: "1.5V"
- note removed: "11 - 12 53VAC 12 - 13 46VAC 13 - 14 3VAC 14 - 15 34VAC 15 - 16 24VAC 11 - 13 6.7VAC 11 - 14 0.7VAC 11 - 15 45VAC 11 - 16 60VAC 12 - 14 59VAC 12 - 15 82VAC 12 - 16 94VAC 13 - 15 49VAC 14 - 16 57VAC 14 - 16 45VAC"
- note removed: "11.2VAC"
- note removed: "12.5V"
- note removed: "13.0V"
- note removed: "187V"
- note removed: "26.1V"
- note removed: "26.3V"
- note removed: "26.5V"
- note removed: "31.6VAC"
- note removed: "32.6V 2.5VAC"
- note removed: "4.4V"
- note removed: "4.6VAC"
- note removed: "44.8VAC"
- note removed: "6.1VAC"
- note removed: "7 - 7.5 6VAC 7.5 - 8 45VAC 7.5 - 9 3VAC 8 - 9 55VAC 9 - 10 1207VAC 7 - 8 33VAC 7 - 9 9VAC 8 - 10 739VAC 7.5 - 10 1208VAC 7 - 10 1174VAC"
- note removed: "7.8V"
- note removed: "71.5V"
- note removed: "71V"
- note removed: "8.2V"
- note removed: "9.6VAC"
- note removed: "TODO: Is this 24V?"
- note removed: "TODO: Is this Z horizontal?"
- note removed: "TODO: Measure voltages around B+ ADJ"
- note removed: "TODO: Renumber PINS??"
- note removed: "TODO: verify voltages"
- moved on the sheet: C101, C102, C103, C104, C105, C106, C107, C109, C110, C111, C112, C114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

Commit message: Added final power filter PCB
Parts:
- added C871, C874: C, Resistor_THT:R_Axial_Power_L20.0mm_W6.4mm_P25.40mm, symbol Device:C
- added C872, C873: C, Capacitor_THT:C_Axial_L3.8mm_D2.6mm_P10.00mm_Horizontal, symbol Device:C
- added COIL_L871: Degauss, symbol Device:L
- added CRT_GND1, WIRE_P3: Conn_01x01_Socket, symbol Connector:Conn_01x01_Socket
- added F871: 250V 3A, Fuse:Fuseholder_Clip-6.3x32mm_Littelfuse_102071_Inline_P34.70x7.60mm_D2.00mm_Horizontal, symbol Device:Fuse
- added J871: Jumper_2_Bridged, _my-footprints:_Jumper_20mm, symbol Jumper:Jumper_2_Bridged
- added L873, L875: L_Coupled, _my-footprints:_choke-pwr-board, symbol Device:L_Coupled
- added P1_P2: IN PUT, _my-footprints:-Connector_01x02XP10.0mm, symbol Connector:Conn_01x02_Pin
- added P3: Conn_01x01_Pin, _my-footprints:-SolderWire, symbol Connector:Conn_01x01_Pin
- added PWR_CN10: L871, _my-footprints:-Connector_01x02XP10.0mm, symbol Connector:Conn_01x02_Pin
- added PWR_CN11: SW871, _my-footprints:-Connector_01x02XP10.0mm, symbol Connector:Conn_01x02_Pin
- added PWR_CN9: Conn_01x03_Pin, _my-footprints:-Connector_01x03, symbol Connector:Conn_01x03_Pin
- added PWR_SW871: Power Switch, symbol Switch:SW_SPST
- added R871: Thermistor_PTC, Resistor_THT:R_Box_L13.0mm_W4.0mm_P9.00mm, symbol Device:Thermistor_PTC
- added R872: R, Resistor_THT:R_Axial_DIN0207_L6.3mm_D2.5mm_P15.24mm_Horizontal, symbol Device:R
- added SH2: RFShield_OnePiece, RF_Shielding:Laird_Technologies_BMI-S-103_26.21x26.21mm, symbol Device:RFShield_OnePiece
- added WIRE_CN10, WIRE_CN11: Conn_01x02_Socket, symbol Connector:Conn_01x02_Socket
- added WIRE_CN9: Conn_01x03_Socket, symbol Connector:Conn_01x03_Socket
- CN9: value Conn_01x01_Pin -> Conn_01x02_Pin
- renumbered JP206 to J206, JP207 to J207, JP502 to J502
Connections:
- net GNDREF: now also G_CN9.3 (GRN); no longer G_CN9.1 (BLK)
- new net: C871.1, L873.3, PWR_CN11.2 (Pin_2)
- new net: C871.2, L873.1, PWR_CN9.2 (WHT), R871.2
- new net: PWR_CN10.1 (Pin_1), PWR_CN11.1 (Pin_1), PWR_CN9.1 (BLK)
- new net: PWR_CN10.2 (Pin_2), R871.1
- new net: C874.2, J871.1 (A), L873.2, L875.1, R872.2
- new net: C872.2, C874.1, L873.4, L875.3, R872.1
- new net: L875.2, P1_P2.1 (WHT)
- new net: F871.2, L875.4
- new net: C872.1, C873.2, P3.1 (GND), PWR_CN9.3 (GRN)
- new net: SH2.1 (PWR_PCB_MOUNT), WIRE_P3.1 (Pin_1)
- new net: COIL_L871.1, WIRE_CN10.1 (Pin_1)
- new net: COIL_L871.2, WIRE_CN10.2 (Pin_2)
- new net: F871.1, P1_P2.2 (BLK)
- new net: PWR_SW871.1 (A), WIRE_CN11.1 (Pin_1)
- new net: PWR_SW871.2 (B), WIRE_CN11.2 (Pin_2)
- new net: C873.1, J871.2 (B)
- new net CRT_GND: CRT1.0 (GND), CRT_GND1.1 (Pin_1)
Other:
- note added: "CHROMA / LUMINANCE"
- note added: "DEFLECTION"
- note added: "JUMPER SANDBOX"
- note added: "PWB-PWR FILTER POWER FILTER PCB"
- note added: "PWR SWITCH PCB"
- note added: "Report any corrections to fredsa@gmail.com If you found this schematic helful, please send an me email to let me know how it went."
- note added: "TEXT/GFX SWITCH PCB"
- note added: "VIDEO AMPLICATION"
- note added: "VIDEO SIGNAL PROCESSING"
- note added: "X-RAY PROTECTION"
- note removed: "32V 60VAC"
- note removed: "79V 61VAC"
- note removed: "Chroma / luminance"
- note removed: "Composite video in"
- note removed: "Deflection"
- note removed: "Jumper sandbox"
- note removed: "Signal processing"
- note removed: "Text/Gfx switch PCB"
- note removed: "X-ray protection"
- moved on the sheet: C103, C135, C136, C138, C139, C140, C161, C205, C207, C208, C209, C210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

Commit message: checkpoint
Parts:
- C871, C874: value C -> .22µF
- C872, C873: value C -> 10nF
- R872: value R -> 330kΩ
Other:
- moved on the sheet: C872, C874, J871, R872

Commit message: checkpoint
Parts:
- added NT5, NT6, NT7, NT8: NetTie, symbol Device:NetTie_2
- NECK_SH1: value RFShield_OnePiece -> Metal Shield
- renumbered CRT1 to CRT_H_9
Connections:
- net BK: now also CRT_H_9.11 (BK)
- net CRT_GND: now also NT5.2, NT7.1; no longer CRT_H_9.0 (GND)
- net FOCUS: now also CRT_H_9.1 (FOCUS)
- net GK: now also CRT_H_9.6 (GK)
- net GND1: no longer C907.2, CN42.2 (G), CN42.3 (G), CN42.5 (G), CN42.9 (H), NECK_CN16.1 (Pin_1)
- net GNDREF: now also NT6.2; no longer G_CN9.3 (GRN)
- net RK: now also CRT_H_9.8 (RK)
- net SCREEN: now also CRT_H_9.7 (S)
- net CRT_10: now reaches CN42.10 (H), R923.2
- net CRT_10: now also CRT_H_9.10 (H)
- net CRT_G: now reaches CRT_H_9.2 (G)
- net CRT_G: now also CRT_H_9.3 (G), CRT_H_9.5 (G)
- net CRT_9: now reaches CRT_H_9.9 (H)
- net CRT_9: now also CN42.9 (H), NT8.2
- net PWR_BLK: now reaches C502.1, C504.2, CN9.1 (BLK), D501.1
- net PWR_BLK: now also WIRE_CN9.1 (BLK)
- net PWR_WHT: now reaches C503.1, C505.2, CN9.2 (WHT), D501.4
- net PWR_WHT: now also WIRE_CN9.2 (WHT)
- net PWR_GRN: now reaches WIRE_CN9.3 (GRN)
- net PWR_GRN: now also G_CN9.3 (GRN), NT6.1
- net B: no longer names the net of C140.1, CN8.1 (B), D107.1 (K)
- net H: no longer names the net of CN8.2 (H), R919.2, R924.2
- new net GND2: C907.2, CN42.2 (G), CN42.3 (G), CN42.5 (G), CRT_H_9.0 (GND), NECK_CN16.1 (Pin_1), NT5.1, NT7.2, NT8.1
Other:
- moved on the sheet: C502, C503, C504, C505, C506, C513, C901, C902, C903, C904, C905, C906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

Commit message: checkpoint
Parts:
- removed NT8: NetTie, symbol Device:NetTie_2
- renumbered JP307 to J307
Connections:
- net CRT_G: now also CRT_H_9.9 (H)
- net GND2: now also CN42.9 (H)
- removed net CRT_9: CN42.9 (H), CRT_H_9.9 (H)
Other:
- moved on the sheet: C222, C223, C224, C229, C230, C513, C901, C902, C903, C904, C905, C906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

Commit message: Cleanup
Other:
- note removed: "0.5V"
- note removed: "0.6V"
- note removed: "0V 9.0VAC"
- note removed: "1.1V"
- note removed: "1.3V"
- note removed: "11.0V"
- note removed: "12.2V"
- note removed: "12.3V"
- note removed: "12.4V"
- note removed: "12.7V"
- note removed: "12.8V"
- note removed: "12.9V"
- note removed: "13.3V"
- note removed: "17.3V"
- note removed: "17.6V"
- note removed: "17.6V 0.7VAC"
- note removed: "18.4V"
- note removed: "2.1V 1.4VAC"
- note removed: "24.9V"
- note removed: "28.1V"
- note removed: "3.4V"
- note removed: "3.6V"
- note removed: "4.3V"
- note removed: "4.4V 4VAC"
- note removed: "4.7V"
- note removed: "4.7V 0.6VAC"
- note removed: "4.9V"
- note removed: "46VAC"
- note removed: "5.1V"
- note removed: "6.3V"
- note removed: "7.3V"
- note removed: "7.9V"
- note removed: "8.0V"
- note removed: "8.4V"
- note removed: "8.5V"
- note removed: "8.9V"
- note removed: "88.7V"
- note removed: "9.0V"
- note removed: "9.2V"
- note removed: "TODO: Define Z ?"
- moved on the sheet: C139, C205, C207, C208, C209, C210, C211, C214, C218, C228, C304, C308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

Commit message: checkpoint
Parts:
- removed NT6: NetTie, symbol Device:NetTie_2
- added TP90: Conn_01x01_Pin, Connector_Pin:Pin_D1.0mm_L10.0mm, symbol Connector:Conn_01x01_Pin
Connections:
- net PWR_GRN is gone; now on net GNDREF: G_CN9.3 (GRN), WIRE_CN9.3 (GRN)
- net VCOM: now also TP90.1 (Pin_1)
Other:
- note added: "-0.01V 43V Pk-Pk 15.7kHz"
- note added: "-10V 186VAC 60Hz 5VAC 15.7kHz"
- note added: "-30V 9.0V Pk-Pk 15.7kHz"
- note added: "-81V 184VAC 60Hz"
- note added: "0.0V 7.9VAC 15.7kHz"
- note added: "0.1V 0.6VAC 15.7kHz"
- note added: "0.3V 0.08 Pk-Pk"
- note added: "0.3V 0.8 Pk-Pk"
- note added: "0.3V 1.0V Pk-Pk"
- note added: "0.3V 1.4V Pk-Pk"
- note added: "0.9V 137VAC 15.7kHz"
- note added: "1.2V 0.3 Pk-Pk"
- note added: "1.2V 7.8VAC 15.7kHz"
- note added: "11.1V 1.2 Pk-Pk"
- note added: "13.3V 0.4VAC"
- note added: "3.3V 1.1 Pk-Pk"
- note added: "3.4V 0.4 Pk-Pk"
- note added: "3.4V 1V Pk-Pk"
- note added: "4.5V 3.0 Pk-Pk"
- note added: "4.8 - 5.6V (COLOR ADJ) 0.4V (TEXT SWITCH) 0.4VAC"
- note added: "6.5V 2.0V Pk-Pk"
- note added: "78V 188VAC 60Hz"
- note added: "79V 188VAC 60Hz"
- note removed: "-0.1V 4VAC"
- note removed: "-1V 144VAC"
- note removed: "-1V 46VAC"
- note removed: "-9V 61VAC"
- note removed: "0.3V"
- note removed: "0.3V 1.9VAC"
- note removed: "0.3V 2.2VAC"
- note removed: "1.2V"
- note removed: "1.8V 4.0VAC"
- note removed: "108V 1670VAC"
- note removed: "13.4V"
- note removed: "158V"
- note removed: "29.1V 16VAC"
- note removed: "31V 80VAC"
- note removed: "4.5V"
- note removed: "80V 61VAC"
- note removed: "TODO: Here GRDPWR//GND_COM ??"
- note removed: "TODO: Measure voltages due to 1) color knob, 2) text switch"
- moved on the sheet: C101, C103, C114, C122, C135, C136, C138, C139, C140, C201, C202, C203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
