File: KiCad/apple-color-monitor-iie-a2m2056/apple-color-monitor-iie-a2m2056.kicad_sch (KiCad schematic)
At the start: 470 parts, among them CN14 Conn_01x04_Pin, CN16 Conn_01x01_Pin, CN20 Conn_01x06_Pin, CN20_plug1 Conn_01x06, CN4 Conn_01x07_Pin, CN4_FRONT1 CN, CN5 Text/Gfx, CN5_FRONT1 Conn_01x02_Socket, CN8 Conn_01x02_Pin, CN9 Conn_01x02_Pin, IC102 CD4053B, J101 Jumper_2_Bridged, J102 Jumper_2_Bridged, J103 Jumper_2_Bridged, J104 Jumper_2_Bridged, J106 Jumper_2_Bridged, J107 Jumper_2_Bridged, J108 Jumper_2_Bridged, J109 Jumper_2_Bridged, J110 Jumper_2_Bridged, J111 Jumper_2_Bridged, J112 Jumper_2_Bridged, J113 Jumper_2_Bridged, J114 Jumper_2_Bridged, J201 Jumper_2_Bridged, J202 Jumper_2_Bridged, J203 Jumper_2_Bridged, J204 Jumper_2_Bridged, J205 Jumper_2_Bridged, J206 Jumper_2_Bridged, J207 Jumper_2_Bridged, J302 Jumper_2_Bridged, J304 Jumper_2_Bridged, J306 Jumper_2_Bridged, J307 Jumper_2_Bridged, J308 Jumper_2_Bridged, J401 Jumper_2_Bridged, J402 Jumper_2_Bridged, J502 Jumper_2_Bridged, J603 Jumper_2_Bridged, J604 Jumper_2_Bridged, J801 Jumper_2_Bridged, J802 Jumper_2_Bridged, J803 Jumper_2_Bridged, J804 Jumper_2_Bridged, J805 Jumper_2_Bridged, J806 Jumper_2_Bridged, J871 Jumper_2_Bridged, J901 Jumper_2_Bridged, P1_P2 IN PUT, P3 Conn_01x01_Pin, P701 VIDEO IN, Q101 C945, Q102 A733, Q103 A733, Q104 C945, Q105 A733, Q111 A642, Q114 C945, Q201 C1507, Q202 D1398, Q501 A709, Q502 C1008, Q503 C3042, Q504 A709, Q801 C945, Q802 C945, Q803 C945, Q804 A733, Q805 A733, Q806 A733, Q807 A733, Q808 A733, Q809 A733, Q901 C1507, Q902 C1507, Q903 C1507, Q904 C2330, Q905 C2330, Q906 C2330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

Commit message: checkpoint
Other:
- note added: "-0.5V 11VAC 15.7kHz"
- note added: "-9V 240VAC 15.7kHZ"
- note added: "0.7V 1.1VAC 60Hz+15.7kHz"
- note added: "1.2V 15.2VAC 60Hz"
- note added: "1.7V 27VAC 60Hz"
- note added: "26.6V 29VAC 60Hz"
- note added: "26V 0.8VAC 15.7kHz"
- note added: "26V 2.4VAC 60Hz"
- note added: "8.3V 7.0VAC 60Hz+15kHz"
- note added: "8.5V 3.5VAC 60Hz+15kHz"
- note added: "8.5V 7.6VAC 60Hz+15kHz"
- note removed: "-3.4V 244VAC 19-20kHZ"
- note removed: "0.6V 2.3VAC"
- note removed: "0.8V 17.6VAC 60Hz"
- note removed: "1.5V 30VAC 60Hz"
- note removed: "24.4V 8VAC"
- note removed: "26.7V 32VAC 60Hz"
- note removed: "8.2V 4.8VAC"
- note removed: "8.2V 7.8VAC 60Hz+15kHz"
- note removed: "8.3V 8.8VAC"
- note removed: "8.4V 8.4VAC 60Hz+15kHz"
- moved on the sheet: D204, D301, R152, R153, R236

Commit message: checkpoint
Other:
- note added: "-0.7V 176VAC 15.7kHz"
- note added: "-1.1V 176VAC 15.7kHz"
- note added: "13.5V 0.8VAC"
- note added: "18.5V 1.2VAC 60Hz"
- note removed: "-1.5V 170VAC ~16kHz"
- note removed: "-5V 170VAC 31.4kHz"
- note removed: "12.3V 6VAC"
Changed lines of the file:
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@@
 		)
 	)
-	(text "17V\n4VAC"
+	(text "18.5V\n1.2VAC\n60Hz"
 		(exclude_from_sim no)
 		(at 340.36 257.81 0)
@@
 		)
 	)
-	(text "12.3V\n6VAC"
+	(text "13.5V\n0.8VAC"
 		(exclude_from_sim no)
-		(at 367.03 258.064 0)
+		(at 367.03 257.81 0)
 		(effects
 			(font
@@
 		)
 	)
-	(text "-1.5V\n170VAC\n~16kHz"
+	(text "-1.1V\n176VAC\n15.7kHz"
 		(exclude_from_sim no)
-		(at 323.7099 257.2509 0)
+		(at 323.85 256.54 0)
 		(effects
 			(font
@@
 		)
 	)
-	(text "-5V\n170VAC\n31.4kHz"
+	(text "-0.7V\n176VAC\n15.7kHz"
 		(exclude_from_sim no)
 		(at 312.42 257.302 0)
@@
 	)
 	(junction
-		(at 337.82 259.08)
-		(diameter 0)
-		(color 0 0 0 0)
-	)
-	(junction
 		(at 383.54 365.76)
 		(diameter 0)
@@
 	)
 	(junction
+		(at 336.55 259.08)
+		(diameter 0)
+		(color 0 0 0 0)
+	)
+	(junction
 		(at 478.79 261.62)
 		(diameter 0)
@@
 	(wire
 		(pts
+			(xy 336.55 259.08) (xy 332.74 259.08)
+		)
+		(stroke
+			(width 0)
+			(type default)
+		)
+	)
+	(wire
+		(pts
 			(xy 434.34 88.9) (xy 430.53 88.9)
 		)
@@
 	(wire
 		(pts
-			(xy 337.82 259.08) (xy 342.9 259.08)
-		)
-		(stroke
-			(width 0)
-			(type default)
-		)
-	)
-	(wire
-		(pts
 			(xy 516.89 261.62) (xy 516.89 250.19)
 		)
@@
 	(wire
 		(pts
+			(xy 336.55 259.08) (xy 342.9 259.08)
+		)
+		(stroke
+			(width 0)
+			(type default)
+		)
+	)
+	(wire
+		(pts
 			(xy 191.77 38.1) (xy 191.77 92.71)
 		)
@@
 	(wire
 		(pts
-			(xy 337.82 259.08) (xy 332.74 259.08)
-		)
-		(stroke
-			(width 0)
-			(type default)
-		)
-	)
-	(wire
-		(pts
 			(xy 36.83 224.79) (xy 16.51 224.79)
 		)
@@
 	(symbol
 		(lib_id "power:PWR_FLAG")
-		(at 337.82 259.08 0)
+		(at 336.55 259.08 0)
 		(unit 1)
 		(body_style 1)
@@
 		(fields_autoplaced yes)
 		(property "Reference" "#FLG06"
-			(at 337.82 257.175 0)
+			(at 336.55 257.175 0)
 			(hide yes)
 			(show_name no)
@@
 		)
 		(property "Value" "PWR_FLAG"
-			(at 337.82 254 0)
+			(at 336.55 254 0)
 			(show_name no)
 			(do_not_autoplace no)
@@
 		)
 		(property "Footprint" ""
-			(at 337.82 259.08 0)
+			(at 336.55 259.08 0)
 			(hide yes)
 			(show_name no)
@@
 		)
 		(property "Datasheet" ""
-			(at 337.82 259.08 0)
+			(at 336.55 259.08 0)
 			(hide yes)
 			(show_name no)
@@
 		)
 		(property "Description" "Special symbol for telling ERC where power comes from"
-			(at 337.82 259.08 0)
+			(at 336.55 259.08 0)
 			(hide yes)
 			(show_name no)

Commit message: checkpoint
Other:
- note added: "-0.4V 1.6VAC 60Hz"
- note added: "-0V 28.8VAC 15.7kHZ"
- note added: "-1.0V (!?)"
- note added: "-1.3V 13.3VAC 60Hz"
- note added: "-2.0V 9.6VAC 60Hz"
- note added: "-2.4V 5.2VAC"
- note added: "-2V 224VAC 15.7kHZ"
- note added: "0.1V 51VAC 60Hz"
- note added: "0.4V 27VAC 60Hz+15.7kHz"
- note added: "0.5V 1.7VAC 60Hz"
- note added: "0.7V 1.6VAC 60Hz"
- note added: "0.7V 1.8VAC 60Hz"
- note added: "0.9V"
- note added: "0V 0.6VAC 60Hz"
- note added: "0V 24VAC 15.7kHZ"
- note added: "0V 27VAC 60Hz+15.7kHz"
- note added: "1.1V 50.4VAC 60Hz"
- note added: "1.4V 9.6VAC"
- note added: "10V 22.4VAC 60Hz"
- note added: "11.0V 0.8VAC 3.6MHz triangle"
- note added: "11.0V 0.8VAC 60Hz sawtooth"
- note added: "11.0V 1.6VAC 3.6MHz triangle"
- note added: "11.3V"
- note added: "11.8V 0.1VAC"
- note added: "13.2V 1.6VAC"
- note added: "150V"
- note added: "18.4V"
- note added: "186V"
- note added: "189V 1VAC"
- note added: "18V 2.4VAC"
- note added: "2.3V"
- note added: "25.0V"
- note added: "26.2V"
- note added: "3.0V 2.6VAC 60Hz sawtooth"
- note added: "3.3V"
- note added: "3.7V"
- note added: "4.0V"
- note added: "4.6V 1.6VAC"
- note added: "5.8V 0.2VAC 3.6MHz sine"
- note added: "5.8V 0.3VAC 3.6MHz sine"
- note added: "8.0V 1.7VAC 60Hz sawtooth"
- note added: "8.2V 1.6VAC"
- note added: "89V"
- note added: "9.0V 1.6VAC"
- note added: "9.1V 1.6VAC"
- note removed: "-0.5V 222VAC 15.7kHZ"
- note removed: "-0.8V 33VAC 60Hz sawtooth"
- note removed: "-0V 24VAC 15.7kHZ"
- note removed: "-0V 28VAC 20kHZ"
- note removed: "-2.2V 10.4VAC"
- note removed: "-2.5V 6.6VAC"
- note removed: "0.2V 4VAC"
- note removed: "0V 29.6VAC 60Hz sawtooth"
- note removed: "11.2V 8.8VAC"
- note removed: "17V 4VAC"
- note removed: "79V"
- moved on the sheet: C121, C124, C125, C126, C304, C307, R141, R143, R144, R158, R161, R213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

Commit message: checkpoint
Connections:
- net +18.4V renamed +18V
Other:
- note added: "0.8V 1.5VAC 15.7kHz"
- note added: "1.5V 1.9VAC 15.7kHz"
- note added: "8.5V 1.3VAC 15.7kHz"
- note removed: "0.7V"
- note removed: "1.4V"
- note removed: "TODO: 18.4 ==> 16V??"
- moved on the sheet: C506, D103, R502, TP90

Commit message: checkpoint
Connections:
- net GNDPWR renamed GHORZ
- net GND_COM renamed GCOM
Other:
- note added: "-0.2V 23V Pk-Pk"
- note added: "-0.2V 30V Pk-Pk 15.7kHz"
- note added: "-0.2V 6V Pk-Pk"
- note added: "-0.4V 1.6V Pk-Pk 60Hz"
- note added: "-0.5V 11V Pk-Pk 15.7kHz"
- note added: "-0.7V 176V Pk-Pk 15.7kHz"
- note added: "-0V 28.8V Pk-Pk 15.7kHZ"
- note added: "-1.1V 176V Pk-Pk 15.7kHz"
- note added: "-1.3V 13.3V Pk-Pk 60Hz"
- note added: "-10V 186V Pk-Pk 60Hz 5V Pk-Pk 15.7kHz"
- note added: "-12V 180V Pk-Pk"
- note added: "-14.5V 344V Pk-Pk 11.5kHz"
- note added: "-2.0V 9.6V Pk-Pk 60Hz"
- note added: "-2.4V 5.2V Pk-Pk"
- note added: "-2V 224V Pk-Pk 15.7kHZ"
- note added: "-4.6V 184V Pk-Pk"
- note added: "-5.0V 184V Pk-Pk"
- note added: "-71V 184V Pk-Pk"
- note added: "-75V 180V Pk-Pk 60Hz"
- note added: "-77.5V 188V Pk-Pk"
- note added: "-78V 208V Pk-Pk 60Hz"
- note added: "-80.5V 188V Pk-Pk"
- note added: "-80V 180V Pk-Pk"
- note added: "-80V 180V Pk-Pk 60Hz"
- note added: "-80V 184V Pk-Pk"
- note added: "-81V 184V Pk-Pk 60Hz"
- note added: "-9V 240V Pk-Pk 15.7kHZ"
- note added: "0.0V 7.9V Pk-Pk 15.7kHz"
- note added: "0.1V"
- note added: "0.1V 0.6V Pk-Pk 15.7kHz"
- note added: "0.1V 51V Pk-Pk 60Hz"
- note added: "0.3V 0.8V Pk-Pk"
- note added: "0.4V 27V Pk-Pk 60Hz+15.7kHz"
- note added: "0.5V 1.7V Pk-Pk 60Hz"
- note added: "0.7V 1.1V Pk-Pk 60Hz+15.7kHz"
- note added: "0.7V 1.6V Pk-Pk 60Hz"
- note added: "0.7V 1.8V Pk-Pk 60Hz"
- note added: "0.8V 1.5V Pk-Pk 15.7kHz"
- note added: "0.8V 8.4V Pk-Pk"
- note added: "0.9V 137V Pk-Pk 15.7kHz"
- note added: "0V 0.6V Pk-Pk 60Hz"
- note added: "0V 24V Pk-Pk 15.7kHZ"
- note added: "0V 27V Pk-Pk 60Hz+15.7kHz"
- note added: "1.1V 1.7V Pk-Pk"
- note added: "1.1V 50V Pk-Pk 60Hz"
- note added: "1.1V 8V Pk-Pk"
- note added: "1.2V"
- note added: "1.2V 0.3V Pk-Pk"
- note added: "1.2V 15V Pk-Pk 60Hz"
- note added: "1.2V 2.2V Pk-Pk"
- note added: "1.2V 7.8V Pk-Pk 15.7kHz"
- note added: "1.3V 2.3V Pk-Pk"
- note added: "1.4V 9.6V Pk-Pk"
- note added: "1.5V 1.9V Pk-Pk 15.7kHz"
- note added: "1.5V 2.6V Pk-Pk"
- note added: "1.7V"
- note added: "1.7V 27V Pk-Pk 60Hz"
- note added: "105V 188V Pk-Pk 60Hz"
- note added: "105V 268V Pk-Pk"
- note added: "105V 300V Pk-Pk"
- note added: "106V 440V Pk-Pk 60Hz + 15.7kHz"
- note added: "10V 22.4V Pk-Pk 60Hz"
- note added: "11.0V 0.8V Pk-Pk 3.6MHz triangle"
- note added: "11.0V 0.8V Pk-Pk 60Hz sawtooth"
- note added: "11.0V 1.6V Pk-Pk 3.6MHz triangle"
- note added: "11.1V 1.2V Pk-Pk"
- note added: "11.8V 0.1V Pk-Pk"
- note added: "115V >900V Pk-Pk 15.7kHz"
- note added: "12.6V 2V Pk-Pk"
- note added: "12.8V 2V Pk-Pk"
- note added: "13.2V 1.6V Pk-Pk"
- note added: "13.3V 0.4V Pk-Pk"
- note added: "13.3V 2V Pk-Pk"
- note added: "13.5V 0.8V Pk-Pk"
- note added: "18.5V 1.2V Pk-Pk 60Hz"
- note added: "187V 0V Pk-Pk"
- note added: "189V 1V Pk-Pk"
- note added: "18V 2.4V Pk-Pk"
- note added: "26.6V 29V Pk-Pk 60Hz"
- note added: "26V 0.8V Pk-Pk 15.7kHz"
- note added: "26V 2.4V Pk-Pk 60Hz"
- note added: "28V"
- note added: "3.0V 2.6V Pk-Pk 60Hz sawtooth"
- note added: "3.3V 1.1V Pk-Pk"
- note added: "3.3V 11.2V Pk-Pk"
- note added: "3.4V 0.4V Pk-Pk"
- note added: "3.5V 3.6V Pk-Pk"
- note added: "3.6V"
- note added: "3.6V 6V Pk-Pk"
- note added: "3.8V"
- note added: "3.9V"
- note added: "4.3V 3.6V Pk-Pk"
- note added: "4.5V 3.0V Pk-Pk"
- note added: "4.6V 1.6V Pk-Pk"
- note added: "4.8 - 5.6V (COLOR ADJ) 0.4V (TEXT SWITCH) 0.4V Pk-Pk"
- note added: "4.8V 188V Pk-Pk"
- note added: "41V"
- note added: "5.8V 0.2V Pk-Pk 3.6MHz sine"
- note added: "5.8V 0.3V Pk-Pk 3.6MHz sine"
- note added: "68.4V 188V Pk-Pk"
- note added: "68V 188V Pk-Pk"
- note added: "69.1V 188V Pk-Pk"
- note added: "69V 188V Pk-Pk"
- note added: "7.6V 2V Pk-Pk"
- note added: "7.7V 2V Pk-Pk"
- note added: "76V 188V Pk-Pk"
- note added: "78V 188V Pk-Pk 60Hz"
- note added: "79V 188V Pk-Pk 60Hz"
- note added: "8.0V 1.7V Pk-Pk 60Hz sawtooth"
- note added: "8.0V 2V Pk-Pk"
- note added: "8.2V 1.6V Pk-Pk"
- note added: "8.3V 7.0V Pk-Pk 60Hz+15kHz"
- note added: "8.5V 1.3V Pk-Pk 15.7kHz"
- note added: "8.5V 3.5V Pk-Pk 60Hz+15kHz"
- note added: "8.5V 7.6V Pk-Pk 60Hz+15kHz"
- note added: "9.0V 1.6V Pk-Pk"
- note added: "9.1V 1.6V Pk-Pk"
- note added: "Soldered on bottom side of PCB"
- note removed: "-0.2V 23VAC"
- note removed: "-0.2V 30VAC 15.7kHz"
- note removed: "-0.2V 6VAC"
- note removed: "-0.4V 1.6VAC 60Hz"
- note removed: "-0.5V 11VAC 15.7kHz"
- note removed: "-0.7V 176VAC 15.7kHz"
- note removed: "-0V 28.8VAC 15.7kHZ"
- note removed: "-1.1V 176VAC 15.7kHz"
- note removed: "-1.3V 13.3VAC 60Hz"
- note removed: "-10V 186VAC 60Hz 5VAC 15.7kHz"
- note removed: "-12V 180VAC"
- note removed: "-14.5V 344VAC 11.5kHz"
- note removed: "-2.0V 9.6VAC 60Hz"
- note removed: "-2.4V 5.2VAC"
- note removed: "-2V 224VAC 15.7kHZ"
- note removed: "-4.6V 184VAC"
- note removed: "-5.0V 184VAC"
- note removed: "-71V 184VAC"
- note removed: "-75V 180VAC 60Hz"
- note removed: "-77.5V 188VAC"
- note removed: "-78V 208VAC 60Hz"
- note removed: "-80.5V 188VAC"
- note removed: "-80V 180VAC"
- note removed: "-80V 180VAC 60Hz"
- note removed: "-80V 184VAC"
- note removed: "-81V 184VAC 60Hz"
- note removed: "-9V 240VAC 15.7kHZ"
- note removed: "-9V 60VAC"
- note removed: "0.0V 7.9VAC 15.7kHz"
- note removed: "0.1V 0.6VAC 15.7kHz"
- note removed: "0.1V 51VAC 60Hz"
- note removed: "0.3V 0.8 Pk-Pk"
- note removed: "0.4V 27VAC 60Hz+15.7kHz"
- note removed: "0.5V 1.7VAC 60Hz"
- note removed: "0.7V 1.1VAC 60Hz+15.7kHz"
- note removed: "0.7V 1.6VAC 60Hz"
- note removed: "0.7V 1.8VAC 60Hz"
- note removed: "0.8V 1.5VAC 15.7kHz"
- note removed: "0.8V 8.4VAC"
- note removed: "0.9V 137VAC 15.7kHz"
- note removed: "0V 0.6VAC 60Hz"
- note removed: "0V 24VAC 15.7kHZ"
- note removed: "0V 27VAC 60Hz+15.7kHz"
- note removed: "0V 5VAC"
- note removed: "1.1V 1.7VAC"
- note removed: "1.1V 50.4VAC 60Hz"
- note removed: "1.1V 8VAC"
- note removed: "1.2V 0.3 Pk-Pk"
- note removed: "1.2V 15.2VAC 60Hz"
- note removed: "1.2V 2.2VAC"
- note removed: "1.2V 7.8VAC 15.7kHz"
- note removed: "1.3V 2.3VAC"
- note removed: "1.4V 9.6VAC"
- note removed: "1.5V 1.9VAC 15.7kHz"
- note removed: "1.5V 2.6VAC"
- note removed: "1.7V 27VAC 60Hz"
- note removed: "105V 188VAC 60Hz"
- note removed: "105V 268VAC"
- note removed: "105V 300VAC"
- note removed: "106V 440VAC 60Hz + 15.7kHz"
- note removed: "108V 60VAC"
- note removed: "10V 22.4VAC 60Hz"
- note removed: "11.0V 0.8VAC 3.6MHz triangle"
- note removed: "11.0V 0.8VAC 60Hz sawtooth"
- note removed: "11.0V 1.6VAC 3.6MHz triangle"
- note removed: "11.1V 1.2 Pk-Pk"
- note removed: "11.8V 0.1VAC"
- note removed: "115V >900VAC 15.7kHz"
- note removed: "12.6V 2VAC"
- note removed: "12.8V 2VAC"
- note removed: "13.2V 1.6VAC"
- note removed: "13.3V 0.4VAC"
- note removed: "13.3V 2VAC"
- note removed: "13.5V 0.8VAC"
- note removed: "18.5V 1.2VAC 60Hz"
- note removed: "187V 0VAC"
- note removed: "189V 1VAC"
- note removed: "18V 2.4VAC"
- note removed: "26.6V 29VAC 60Hz"
- note removed: "26V 0.8VAC 15.7kHz"
- note removed: "26V 2.4VAC 60Hz"
- note removed: "3.0V 2.6VAC 60Hz sawtooth"
- note removed: "3.3V 1.1 Pk-Pk"
- note removed: "3.3V 11.2VAC"
- note removed: "3.4V 0.4 Pk-Pk"
- note removed: "3.5V 3.6VAC"
- note removed: "3.6V 6VAC"
- note removed: "4.3V 3.6VAC"
- note removed: "4.5V 3.0 Pk-Pk"
- note removed: "4.6V 1.6VAC"
- note removed: "4.8 - 5.6V (COLOR ADJ) 0.4V (TEXT SWITCH) 0.4VAC"
- note removed: "4.8V 188VAC"
- note removed: "5.8V 0.2VAC 3.6MHz sine"
- note removed: "5.8V 0.3VAC 3.6MHz sine"
- note removed: "68.4V 188VAC"
- note removed: "68V 188VAC"
- note removed: "69.1V 188VAC"
- note removed: "69V 188VAC"
- note removed: "7.6V 2VAC"
- note removed: "7.7V 2VAC"
- note removed: "76V 188VAC"
- note removed: "78V 188VAC 60Hz"
- note removed: "79V 188VAC 60Hz"
- note removed: "79V 60VAC"
- note removed: "8.0V 1.7VAC 60Hz sawtooth"
- note removed: "8.0V 2VAC"
- note removed: "8.2V 1.6VAC"
- note removed: "8.3V 7.0VAC 60Hz+15kHz"
- note removed: "8.5V 1.3VAC 15.7kHz"
- note removed: "8.5V 3.5VAC 60Hz+15kHz"
- note removed: "8.5V 7.6VAC 60Hz+15kHz"
- note removed: "9.0V 1.6VAC"
- note removed: "9.1V 1.6VAC"
- note removed: "TODO: Zener?"
- note removed: "TODO: describe as +170V ??"
- note removed: "TODO: describe as +50V ??"
- moved on the sheet: C117, C201, C202, C203, C204, C213, C220, C222, C227, C228, C508, C514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

Commit message: checkpoint
Other:
- note added: "-0.2V 6.2V RMS / 22V Pk-Pk 15.7kHz"
- note added: "-2V 36V RMS / 140V Pk-Pk 15.7kHz"
- note added: "157V 28V Pk-Pk 60Hz"
- note added: "3.4V 4.4V RMS / 10V Pk-Pk 15.7kHz"
- note added: "3.6V 3.6V RMS / 2.3V Pk-Pk 15.7kHz"
- note added: "3.7V 4.0V RMS / 5.5V Pk-Pk 15.7kHz"
- note added: "4.4V 4.4V RMS / 2.6V Pk-Pk 15.7kHz"
- note added: "86V 24V Pk-Pk 60Hz"
- note added: "Please check that you have the latest version of this schematic from: https://github.com/fredsa/apple-color-monitor-iie-a2m2056 Flyback and other transformer configuration may be drawn incorrectly. Report any corrections to this schematic to: fredsa@gmail.com If you found this schematic helful, please send an me email to let me know how it went."
- note removed: "-0.2V 23V Pk-Pk"
- note removed: "0.9V 137V Pk-Pk 15.7kHz"
- note removed: "3.3V 11.2V Pk-Pk"
- note removed: "3.5V 3.6V Pk-Pk"
- note removed: "3.6V 6V Pk-Pk"
- note removed: "4.3V 3.6V Pk-Pk"
- note removed: "7.6V 2V Pk-Pk"
- note removed: "7.7V 2V Pk-Pk"
- note removed: "Report any corrections to fredsa@gmail.com If you found this schematic helful, please send an me email to let me know how it went."
- moved on the sheet: C118, C130, C138, C218, C512, D202, D207, D301, D503, D508, R125, R230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

Commit message: neck board cleanup
Other:
- note removed: "1.2V 2.2V Pk-Pk"
- moved on the sheet: C901, C902, C903, C904, C905, C906, C907, C908, CN42, CRT_ANODE1, CRT_H_9, J901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

Commit message: Updated comments
Other:
- note added: "Please check that you have the latest version of this schematic from: https://github.com/fredsa/apple-color-monitor-iie-a2m2056 Flyback and other transformer configurations may be drawn incorrectly. Report any corrections to this schematic to: fredsa@gmail.com I've spent many hours recreating this schematic. If you found this schematic to be helful, please send me an email to let me know how it w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"
- note removed: "Please check that you have the latest version of this schematic from: https://github.com/fredsa/apple-color-monitor-iie-a2m2056 Flyback and other transformer configuration may be drawn incorrectly. Report any corrections to this schematic to: fredsa@gmail.com If you found this schematic helful, please send an me email to let me know how it went."
Changed lines of the file:
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@@
 		)
 	)
-	(text "Please check that you have the latest version of this schematic from:\nhttps://github.com/fredsa/apple-color-monitor-iie-a2m2056\n\nFlyback and other transformer configuration may be drawn incorrectly.\nReport any corrections to this schematic to: fredsa@gmail.com\n\nIf you found this schematic helful, please send an me email to let me know how it went."
+	(text "Please check that you have the latest version of this schematic from:\nhttps://github.com/fredsa/apple-color-monitor-iie-a2m2056\n\nFlyback and other transformer configurations may be drawn incorrectly.\nReport any corrections to this schematic to: fredsa@gmail.com\n\nI've spent many hours recreating this schematic. If you found this schematic\nto be helful, please send me an email to let me know how it went.\n\nVoltages are shown as measured, but may not represent correct factory\ncalibration due to incorrect adjustments made by a previous owner."
 		(exclude_from_sim no)
-		(at 525.272 368.3 0)
+		(at 525.272 363.474 0)
 		(effects
 			(font
